File: MainBoard_Relay/MainBoard_Relay.kicad_pcb (KiCad board)
At the start: 2 copper layers, 49.2 x 41.6 mm, 27 parts, among them J1 Conn_01x03_Female, J2 Conn_01x03_Female, K1 G5Q-1, K2 RAC01-05SGB, Q1 Q_NMOS_DGS, U1 ESP-01v090, U2 AZ1117-3.3

Commit message: RGB and Relay platform finished
Parts:
- C1, C2: value C -> 1uF
- moved REF** 6.84 mm to (169.3, 79.6)
- moved REF** 3.30 mm to (180.7, 79.8)
- moved REF** 3.18 mm to (175.6, 70.6)
- moved REF** 2.91 mm to (161.6, 79.5)
- moved R1 2.26 mm to (154.5, 66.5), turned to 0 degrees
- moved REF** 1.92 mm to (187.5, 76.9)
- moved D1 1.24 mm to (154.5, 64.6), turned to 0 degrees
Connections:
- net Net-(J1-Pad2) renamed /ACN
- J1 pad 3: Net-(J1-Pad3) -> /ACL
- K1 pad 1: +5V -> /ACL
- K1 pad 2: Net-(J1-Pad3) -> Net-(K1-Pad2)
- K1 pad 5: Net-(K1-Pad5) -> +5V
- K2 pad 1: Net-(J1-Pad3) -> /ACL
- Q1 pad 1: Net-(K1-Pad5) -> Net-(K1-Pad2)
- U2 pad 4: GND -> (no net)
Routing:
- net /ACL: track 0.00 -> 54.5 mm
- net Net-(J1-Pad3): track 45.2 -> 0.00 mm
- net /ACN: track 62.5 -> 23.9 mm
- net Net-(K1-Pad5): track 37.7 -> 0.00 mm, vias 1 -> 0
- net Net-(K1-Pad2): track 0.00 -> 22.5 mm
- net +5V: track 83.1 -> 89.7 mm
- net Net-(D1-Pad2): track 2.80 -> 1.90 mm
- added copper zone on F.Cu, net /ACN
